File: PowerBank_KICAD/_autosave-OZE_PowerBank.kicad_sch (KiCad schematic)
At the start: 84 parts, among them IC1 TPS2514ADBVT, IC3 TPS25810RVCR, J1 Conn_01x02_Pin, J10 Conn_01x04_Pin, J11 Conn_01x02_Pin, J12 Battery with BMS Input, J2 DCJ200-10-A-XX-K_REVA, J3 Conn_01x04_Pin, J4 Conn_01x04_Pin, J5 Conn_01x04_Pin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

Commit message: zmieniony symbol biblioteczny TPS, dodano footprinty, zmieniono piny wyprowadzeniowe, dodano opis funkci pinów STM , konfiguracja kanalow ADC
Parts:
- SW2: footprint (none) -> LIB_SLW-1276864-4A-D:SLW12768644AD
Changed lines of the file:
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@@
 			)
 		)
-		(property "Footprint" ""
+		(property "Footprint" "LIB_SLW-1276864-4A-D:SLW12768644AD"
 			(at 96.52 294.64 0)
 			(effects
